File: vco1_components.sch (EAGLE design)
At the start: 56 parts, among them IC1 LM13700N, Q3 2N3904, Q4 2N3904, U1 TL072_, U2 TL072_, U3 TL072_

Commit message: Make trimpot accessible from side
...when side-trimmable trimpot ist used.
Parts:
- R10: value 1.2m -> 1.2M
- R3: value 2.2m -> 2.2M

Commit message: Update comment about C3
Thomas Henry proposes to use Polystyrene for low temperature drift, but
there are caps with "0" temperature drift, so let's use these.
Other:
- note added: "Make C3 NP0/C0G"
- note removed: "Make C3 Polystyrene"
Changed lines of the file:
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@@
 <drawing>
 <settings>
-<setting alwaysvectorfont="no"/>
+<setting alwaysvectorfont="yes"/>
 <setting keepoldvectorfont="yes"/>
 <setting verticaltext="up"/>
@@
 In physical contact with 2n3906s
 2N3906s should be epoxied together</text>
-<text x="223.52" y="314.96" size="1.778" layer="91">Make C3 Polystyrene</text>
+<text x="223.52" y="314.96" size="1.778" layer="91">Make C3 NP0/C0G</text>
 <text x="241.3" y="269.24" size="1.778" layer="91">R10 = 1.2m for 12v
 was 1.5m for 15v
